Commit message: 0514

File: my_robot/xacro/my_robot07.xacro (robot description, xacro)
@@ -41,5 +41,5 @@
       <mass value="0.1"/>
       <origin xyz="0 0 0.0625" rpy="0 ${90*pi/180} 0"/>
-      <inertia ixx="1.0" ixy="0.0" ixz="0.0" iyy="1.0" iyz="0.0" izz="1.0"/>
+      <inertia ixx="0.01" ixy="0.0" ixz="0.0" iyy="0.01" iyz="0.0" izz="0.01"/>
     </inertial>
     <visual>
@@ -95,5 +95,5 @@
       <mass value="0.1"/>
       <origin xyz="-0.09 0 0.2" rpy="0 0 0"/>
-      <inertia ixx="1.0" ixy="0.0" ixz="0.0" iyy="1.0" iyz="0.0" izz="1.0"/>
+      <inertia ixx="0.01" ixy="0.0" ixz="0.0" iyy="0.01" iyz="0.0" izz="0.01"/>
     </inertial>
     <visual>
@@ -114,7 +114,8 @@
     <material>Gazebo/Orange</material>
   </gazebo>
-  <joint name="arm2_joint" type="continuous">
+  <joint name="arm2_joint" type="revolute">
     <parent link="arm2_joint_link"/>
     <child link="arm2_link"/>
+    <limit upper="0.0" lower="-0.7" effort="100" velocity="100"/>
     <axis xyz="0 1 0"/>
     <origin xyz="-0.09 0 0.2" rpy="0 0 0"/>
@@ -139,5 +140,5 @@
       <mass value="0.08"/>
       <origin xyz="-0.014953 0 0.073494" rpy="0 ${-11.5*pi/180} 0"/>
-      <inertia ixx="1.0" ixy="0.0" ixz="0.0" iyy="1.0" iyz="0.0" izz="1.0"/>
+      <inertia ixx="0.01" ixy="0.0" ixz="0.0" iyy="0.01" iyz="0.0" izz="0.01"/>
     </inertial>
     <visual>
@@ -161,5 +162,5 @@
     <parent link="arm2_link"/>
     <child link="arm1_joint_link"/>
-    <limit upper="1.4" lower="0.0" effort="1000" velocity="100"/>
+    <limit upper="1.4" lower="0.0" effort="100" velocity="100"/>
     <axis xyz="0 1 0"/>
     <origin xyz="-0.029906 0.03 0.146988" rpy="0 0 0"/>
@@ -184,5 +185,5 @@
       <origin xyz="0 -0.015 0" rpy="${90*pi/180} 0 0"/>
       <mass value="0.1"/>
-      <inertia ixx="1.0" ixy="0.0" ixz="0.0" iyy="1.0" iyz="0.0" izz="1.0"/>
+      <inertia ixx="0.01" ixy="0.0" ixz="0.0" iyy="0.01" iyz="0.0" izz="0.01"/>
     </inertial>
     <visual>
@@ -211,5 +212,5 @@
       <origin xyz="-0.014953 0 -0.073494" rpy="0 ${11.5*pi/180} 0"/>
       <mass value="0.08"/>
-      <inertia ixx="1.0" ixy="0.0" ixz="0.0" iyy="1.0" iyz="0.0" izz="1.0"/>
+      <inertia ixx="0.01" ixy="0.0" ixz="0.0" iyy="0.01" iyz="0.0" izz="0.01"/>
     </inertial>
     <visual>
@@ -238,5 +239,5 @@
       <mass value="0.1"/>
       <origin xyz="-0.029906 0 -0.146988" rpy="0 0 0"/>
-      <inertia ixx="1.0" ixy="0.0" ixz="0.0" iyy="1.0" iyz="0.0" izz="1.0"/>
+      <inertia ixx="0.01" ixy="0.0" ixz="0.0" iyy="0.01" iyz="0.0" izz="0.01"/>
     </inertial>
     <visual>

Commit message: 0516

File: my_robot/xacro/my_robot07.xacro (robot description, xacro)
@@ -93,16 +93,16 @@
   <link name="arm2_joint_link">
     <inertial>
-      <mass value="0.1"/>
-      <origin xyz="-0.09 0 0.2" rpy="0 0 0"/>
-      <inertia ixx="0.01" ixy="0.0" ixz="0.0" iyy="0.01" iyz="0.0" izz="0.01"/>
-    </inertial>
-    <visual>
-      <origin xyz="-0.09 0 0.2" rpy="0 0 0"/>
-      <geometry>
-        <sphere radius="0.015"/>
-      </geometry>
-    </visual>
-    <collision>
-      <origin xyz="-0.09 0 0.2" rpy="0 0 0"/>
+      <mass value="1.5"/>
+      <origin xyz="-0.09 0 0.208819" rpy="0 0 0"/>
+      <inertia ixx="0.01" ixy="0.0" ixz="0.0" iyy="0.01" iyz="0.0" izz="0.01"/>
+    </inertial>
+    <visual>
+      <origin xyz="-0.09 0 0.208819" rpy="0 0 0"/>
+      <geometry>
+        <sphere radius="0.015"/>
+      </geometry>
+    </visual>
+    <collision>
+      <origin xyz="-0.09 0 0.208819" rpy="0 0 0"/>
       <geometry>
         <sphere radius="0.015"/>
@@ -111,5 +111,4 @@
   </link>
   <gazebo reference="arm2_joint_link">
-    <selfCollide>true</selfCollide>
     <material>Gazebo/Orange</material>
   </gazebo>
@@ -117,7 +116,7 @@
     <parent link="arm2_joint_link"/>
     <child link="arm2_link"/>
-    <limit upper="0.0" lower="-0.7" effort="100" velocity="100"/>
+    <limit upper="0.0" lower="-0.7" effort="5" velocity="100"/>
     <axis xyz="0 1 0"/>
-    <origin xyz="-0.09 0 0.2" rpy="0 0 0"/>
+    <origin xyz="-0.09 0 0.208819" rpy="0 0 0"/>
     <dynamics damping="0.1"/>
   </joint>
@@ -156,5 +155,4 @@
   </link>
   <gazebo reference="arm2_link">
-    <selfCollide>true</selfCollide>
     <material>Gazebo/Blue</material>
   </gazebo>
@@ -162,5 +160,5 @@
     <parent link="arm2_link"/>
     <child link="arm1_joint_link"/>
-    <limit upper="1.4" lower="0.0" effort="100" velocity="100"/>
+    <limit upper="1.4" lower="0.0" effort="10" velocity="100"/>
     <axis xyz="0 1 0"/>
     <origin xyz="-0.029906 0.03 0.146988" rpy="0 0 0"/>
@@ -201,5 +199,4 @@
   </link>
   <gazebo reference="arm1_joint_link">
-    <selfCollide>true</selfCollide>
     <material>Gazebo/Orange</material>
   </gazebo>
@@ -228,5 +225,4 @@
   </link>
   <gazebo reference="arm1_link">
-    <selfCollide>true</selfCollide>
     <material>Gazebo/Red</material>
   </gazebo>

File: sim1/urdf/arm_robot.urdf (robot description, URDF)
Before this commit: robot arm_robot, 3 links, 2 joints
Joints:
- joint arm1_joint: limit lower=-1.5 upper=1.5 effort=0 velocity=0 -> lower=-3.14 upper=3.14 effort=50 velocity=100; origin xyz=0 0.1 1.0 rpy=0 1.5708 0 -> xyz=0 0.1 1.0 rpy=0 0 0; type prismatic -> continuous
