Commit message: 20190713

File: my_robot/xacro/my_robot11.xacro (robot description, xacro)
@@ -1,4 +1,4 @@
 <?xml version="1.0"?>
-<!--full-->
+<!--spring-->
 <robot name="my_robot" xmlns:xacro="http://ros.org/wiki/xacro">
   <xacro:property name="pi" value="3.1415926535897931" />
@@ -29,27 +29,13 @@
   <gazebo reference="base_link">
     <selfCollide>true</selfCollide>
-    <material>Gazebo/Gold</material>
+    <material>Gazebo/Gray</material>
   </gazebo>
   <joint name="guide_joint" type="prismatic">
     <parent link="base_link"/>
     <child link="guide_link"/>
-    <limit upper="0.8" lower="0.0" effort="0" velocity="100"/>
-    <origin xyz="0.2 0 0.16481" rpy="0 ${-90*pi/180} 0"/>
+    <limit upper="0.40" lower="-0.16" effort="1000" velocity="100"/>
+    <origin xyz="0.2 0 0.334813" rpy="0 ${-90*pi/180} 0"/>
     <dynamics damping="0.1"/>
   </joint>
-  <transmission name="guide_trans">
-    <type>transmission_interface/SimpleTransmission</type>
-    <joint name="guide_joint">
-      <hardwareInterface>hardware_interface/EffortJointInterface</hardwareInterface>
-    </joint>
-    <actuator name="guide_motor">
-       <hardwareInterface>hardware_interface/EffortJointInterface</hardwareInterface>
-       <mechanismReduction>1</mechanismReduction>
-    </actuator>
-  </transmission>
-  <gazebo reference="guide_joint">
-    <provideFeedback>true</provideFeedback>
-    <turnGravityOff>false</turnGravityOff>
-  </gazebo>
   <link name="guide_link">
     <inertial>
@@ -73,5 +59,5 @@
   <gazebo reference="guide_link">
     <selfCollide>true</selfCollide>
-    <material>Gazebo/Gold</material>
+    <material>Gazebo/Gray</material>
   </gazebo>
   <joint name="hashida_joint" type="fixed">
@@ -131,5 +117,5 @@
     <parent link="arm2_joint_link"/>
     <child link="arm2_link"/>
-    <limit upper="0.0" lower="-0.7" effort="10" velocity="100"/>
+    <limit upper="${35*pi/180}" lower="0.0" effort="5" velocity="100"/>
     <axis xyz="0 1 0"/>
     <origin xyz="-0.09 0 0.208819" rpy="0 0 0"/>
@@ -152,10 +138,10 @@
   <link name="arm2_link">
     <inertial>
-      <mass value="0.2"/>
-      <origin xyz="-0.014953 0 0.073494" rpy="0 ${-11.5*pi/180} 0"/>
-      <inertia ixx="0.01" ixy="0.0" ixz="0.0" iyy="0.01" iyz="0.0" izz="0.01"/>
-    </inertial>
-    <visual>
-      <origin xyz="-0.014953 0 0.073494" rpy="0 ${-11.5*pi/180} 0"/>
+      <mass value="0.1"/>
+      <origin xyz="-0.057453 0 0.048209" rpy="0 ${-50*pi/180} 0"/>
+      <inertia ixx="0.01" ixy="0.0" ixz="0.0" iyy="0.01" iyz="0.0" izz="0.01"/>
+    </inertial>
+    <visual>
+      <origin xyz="-0.057453 0 0.048209" rpy="0 ${-50*pi/180} 0"/>
       <geometry>
         <cylinder length="0.15" radius="0.015"/>
@@ -163,5 +149,5 @@
     </visual>
     <collision>
-      <origin xyz="-0.014953 0 0.073494" rpy="0 ${-11.5*pi/180} 0"/>
+      <origin xyz="-0.057453 0 0.048209" rpy="0 ${-50*pi/180} 0"/>
       <geometry>
         <cylinder length="0.15" radius="0.015"/>
@@ -175,7 +161,7 @@
     <parent link="arm2_link"/>
     <child link="arm1_joint_link"/>
-    <limit upper="1.4" lower="0.0" effort="20" velocity="100"/>
+    <limit upper="0.0" lower="${-70*pi/180}" effort="10" velocity="100"/>
     <axis xyz="0 1 0"/>
-    <origin xyz="-0.029906 0.03 0.146988" rpy="0 0 0"/>
+    <origin xyz="-0.114907 0 0.096418" rpy="0 0 0"/>
     <dynamics damping="0.1"/>
   </joint>
@@ -196,18 +182,18 @@
   <link name="arm1_joint_link">
     <inertial>
-      <origin xyz="0 -0.015 0" rpy="${90*pi/180} 0 0"/>
-      <mass value="0.05"/>
-      <inertia ixx="0.01" ixy="0.0" ixz="0.0" iyy="0.01" iyz="0.0" izz="0.01"/>
-    </inertial>
-    <visual>
-      <origin xyz="0 -0.015 0" rpy="${90*pi/180} 0 0"/>
-      <geometry>
-        <cylinder length="0.06" radius="0.015"/>
-      </geometry>
-    </visual>
-    <collision>
-      <origin xyz="0 -0.015 0" rpy="${90*pi/180} 0 0 "/>
-      <geometry>
-        <cylinder length="0.06" radius="0.015"/>
+      <origin xyz="0 0 0" rpy="${90*pi/180} 0 0"/>
+      <mass value="0.1"/>
+      <inertia ixx="0.01" ixy="0.0" ixz="0.0" iyy="0.01" iyz="0.0" izz="0.01"/>
+    </inertial>
+    <visual>
+      <origin xyz="0 0 0" rpy="${90*pi/180} 0 0"/>
+      <geometry>
+        <cylinder length="0.03" radius="0.015"/>
+      </geometry>
+    </visual>
+    <collision>
+      <origin xyz="0 0 0" rpy="${90*pi/180} 0 0 "/>
+      <geometry>
+        <cylinder length="0.03" radius="0.015"/>
       </geometry>
     </collision>
@@ -222,10 +208,10 @@
   <link name="arm1_link">
     <inertial>
-      <origin xyz="-0.014953 0 -0.073494" rpy="0 ${11.5*pi/180} 0"/>
-      <mass value="0.2"/>
-      <inertia ixx="0.01" ixy="0.0" ixz="0.0" iyy="0.01" iyz="0.0" izz="0.01"/>
-    </inertial>
-    <visual>
-      <origin xyz="-0.014953 0 -0.073494" rpy="0 ${11.5*pi/180} 0"/>
+      <origin xyz="-0.057453 0 -0.048209" rpy="0 ${50*pi/180} 0"/>
+      <mass value="0.08"/>
+      <inertia ixx="0.01" ixy="0.0" ixz="0.0" iyy="0.01" iyz="0.0" izz="0.01"/>
+    </inertial>
+    <visual>
+      <origin xyz="-0.057453 0 -0.048209" rpy="0 ${50*pi/180} 0"/>
       <geometry>
         <cylinder length="0.15" radius="0.015"/>
@@ -233,5 +219,5 @@
     </visual>
     <collision>
-      <origin xyz="-0.014953 0 -0.073494" rpy="0 ${11.5*pi/180} 0"/>
+      <origin xyz="-0.057453 0 -0.048209" rpy="0 ${50*pi/180} 0"/>
       <geometry>
         <cylinder length="0.15" radius="0.015"/>
@@ -248,10 +234,10 @@
   <link name="arm0_link">
     <inertial>
-      <mass value="0.05"/>
-      <origin xyz="-0.029906 0 -0.146988" rpy="0 0 0"/>
-      <inertia ixx="0.01" ixy="0.0" ixz="0.0" iyy="0.01" iyz="0.0" izz="0.01"/>
-    </inertial>
-    <visual>
-      <origin xyz="-0.029906 0 -0.146988" rpy="0 0 0"/>
+      <mass value="0.1"/>
+      <origin xyz="-0.114907 0 -0.096418" rpy="0 0 0"/>
+      <inertia ixx="0.01" ixy="0.0" ixz="0.0" iyy="0.01" iyz="0.0" izz="0.01"/>
+    </inertial>
+    <visual>
+      <origin xyz="-0.114907 0 -0.096418" rpy="0 0 0"/>
       <geometry>
         <sphere radius="0.015"/>
@@ -259,5 +245,5 @@
     </visual>
     <collision>
-      <origin xyz="-0.029906 0 -0.146988" rpy="0 0 0"/>
+      <origin xyz="-0.114907 0 -0.096418" rpy="0 0 0"/>
       <geometry>
         <sphere radius="0.015"/>
@@ -270,4 +256,33 @@
     <selfCollide>true</selfCollide>
     <material>Gazebo/Green</material>
+  </gazebo>
+  <!--spring-->
+  <joint name="spring2_joint" type="prismatic">
+    <parent link="arm2_joint_link"/>
+    <child link="spring_link"/>
+    <limit upper="0.01" lower="0" effort="1000" velocity="100"/>
+    <origin xyz="-0.105 0 0.208819" rpy="0 0 0"/>
+  </joint>
+  <link name="spring_link">
+    <inertial>
+      <origin xyz="-0.0999065 0 0" rpy="0 ${-90*pi/180} 0"/>
+      <mass value="0.001"/>
+      <inertia ixx="0.01" ixy="0.0" ixz="0.0" iyy="0.01" iyz="0.0" izz="0.01"/>
+    </inertial>
+    <visual>
+      <origin xyz="-0.0999065 0 0" rpy="0 ${-90*pi/180} 0"/>
+      <geometry>
+        <cylinder length="0.169813" radius="0.015"/>
+      </geometry>
+    </visual>
+    <collision>
+      <origin xyz="-0.0999065 0 0" rpy="0 ${-90*pi/180} 0"/>
+      <geometry>
+        <cylinder length="0.169813" radius="0.015"/>
+      </geometry>
+    </collision>
+  </link>
+  <gazebo reference="spring_link">
+    <material>Gazebo/Purple</material>
   </gazebo>
   <gazebo>
